Commit message: adding plate to robot

File: spikeball_project/panda_spikeball.urdf (robot description, URDF)
Before this commit: robot panda_collision, 8 links, 7 joints
Links:
- added link plate, mass 0.0001; visual box size=0.5 0.01 0.1
Joints:
- added joint plate_joint: type prismatic, parent link7, child plate, origin xyz=0 0 0.1654 rpy=0 0 -0.78539816339, axis 0 0 1, limit lower=0.0 upper=0.1 effort=2000 velocity=0.1
- joint joint1: origin xyz=0 0 0.333 rpy=0 0 0 -> xyz=0 0 0.333 rpy=0 0 1.5708
- joint joint6: origin xyz=0 0 0 rpy=1.57079632679 0 0 -> xyz=0 0 0 rpy=0 0 0

Commit message: end plate is fixed

File: spikeball_project/panda_spikeball.urdf (robot description, URDF)
Before this commit: robot panda_collision, 9 links, 8 joints
Links:
- link plate: geometry collision box size=0.5 0.01 0.1; visual box size=0.5 0.01 0.1
Joints:
- joint plate_joint: limit lower=0.0 upper=0.1 effort=2000 velocity=0.1 -> (none); type prismatic -> fixed

Commit message: 5.29.1

File: spikeball_project/panda_spikeball.urdf (robot description, URDF)
Before this commit: robot panda_collision, 9 links, 8 joints
Links:
- removed link plate
Joints:
- removed joint plate_joint

Commit message: plate movement and EE position

File: spikeball_project/panda_spikeball.urdf (robot description, URDF)
Before this commit: robot panda_collision, 8 links, 7 joints
Links:
- added link plate, mass 0.0001; collision box size=0.25 0.01 0.25; visual box size=0.25 0.01 0.25
Joints:
- added joint plate_joint: type fixed, parent link7, child plate, origin xyz=0 0 0.1654 rpy=0 0 -0.78539816339, axis 0 0 1

Commit message: More orientation fixes as well as increased ball size

File: spikeball_project/panda_spikeball.urdf (robot description, URDF)
Before this commit: robot panda_collision, 9 links, 8 joints
Links:
- link link0: geometry visual mesh filename=../../../model/panda/meshes/visual/link0.obj
- link link1: geometry visual mesh filename=../../../model/panda/meshes/visual/link1.obj
- link link2: geometry visual mesh filename=../../../model/panda/meshes/visual/link2.obj
- link link3: geometry visual mesh filename=../../../model/panda/meshes/visual/link3.obj
- link link5: geometry visual mesh filename=../../../model/panda/meshes/visual/link5.obj
